File: PCBs/RCU/_autosave-RCU.kicad_pcb (KiCad board)
At the start: 2 copper layers, 155 parts, among them J100 Conn_01x02, J200 USB_C_Receptacle_USB2.0, J201 Conn_01x05, J300 Right_Motor_Screw_Terminal, J301 Right_Encoder_Conn, J302 Left_Motor_Screw_Terminal, J303 Left_Encoder_Conn, J400 USB_C_Receptacle_USB2.0, Q400 2N7002NXAKR (NMOS), Q401 2N7002NXAKR (NMOS), Q402 BSS84AK,215 (PMOS), Q403 2N7002NXAKR (NMOS), SW201 SW_Push, SW400 SW_Push, SW401 SW_SPDT, U100 AP63203WU, U101 AZ1117-3.3, U102 AP63203WU, U103 LM2576S-ADJ, U200 STM32G0B1CBT6, U201 USBLC6-2SC6, U300 OPA320, U301 DRV8876, U302 OPA320, U303 DRV8876, U400 USBLC6-2SC6, U401 CH340C, U402 ESP32-MINI-1, U403 DG2788ADN-T1-GE4, U500 APDS-9306-065, U501 LSM6DS3, U502 SHT30-DIS, U600 ADC121C027CIMK/NOPB, U601 OPA320, U602 ADC121C027CIMK/NOPB, U603 OPA320, U700 SST26VF032BT-104I/SM, Y200 16MHz

Commit message: USB2 can now power all modules except motor control if it is the only power source that is plugged in
Parts:
- removed C113: 100nF, Capacitor_SMD:C_0603_1608Metric
- removed C114, C115: 22uF, Capacitor_SMD:C_0603_1608Metric
- removed C116: 100uF, Capacitor_THT:CP_Radial_D5.0mm_P2.50mm
- removed C117: 1000uF, Capacitor_THT:CP_Radial_D5.0mm_P2.50mm
- removed D105: 1N5822, Diode_THT:D_DO-201AD_P15.24mm_Horizontal
- removed L104: 15uH, Inductor_SMD:L_0603_1608Metric
- removed L105: 68uH, Inductor_SMD:L_12x12mm_H6mm
- removed U103: LM2576S-ADJ, Package_TO_SOT_SMD:TO-263-5_TabPin3
- added C101: 100uF, Capacitor_THT:CP_Radial_D5.0mm_P2.50mm, F.Cu at (254.4, 35.8)
- added L100: 68uH, Inductor_SMD:L_12x12mm_H6mm, F.Cu at (244.9, 39.6)
- C102: value 10uF -> 1000uF; footprint Capacitor_SMD:C_0603_1608Metric -> Capacitor_THT:CP_Radial_D5.0mm_P2.50mm
- C103: value 100nF -> 10uF
- C104: value 22uF -> 100nF
- C106, C110: value 1uF -> 22uF
- C108: value 22uF -> 1uF
- C112: value 10uF -> 1uF
- D100: value SM5817 -> 1N5822; footprint Schottky_Diode:SODFL3719X135N -> Diode_THT:D_DO-201AD_P15.24mm_Horizontal
- L101: value 82uH -> 15uH
- R100: value 5R -> 8.9k
- R101: value 8.9k -> 1.5k
- R102: value 1.5k -> 5R
- U100: value AP63203WU -> LM2576S-ADJ; footprint Package_TO_SOT_SMD:TSOT-23-6 -> Package_TO_SOT_SMD:TO-263-5_TabPin3
- U101: value AZ1117-3.3 -> AP63203WU; footprint Package_TO_SOT_SMD:TO-252-2 -> Package_TO_SOT_SMD:TSOT-23-6
- U102: value AP63203WU -> AZ1117-3.3; footprint Package_TO_SOT_SMD:TSOT-23-6 -> Package_TO_SOT_SMD:TO-252-2
- moved L103 301.6 mm to (-51.0, 133.0)
- moved C111 298.5 mm to (-57.0, 136.0)
- moved C112 295.8 mm to (-45.0, 136.0)
- moved D102 282.8 mm to (-14.0, 182.0)
- moved C107 281.5 mm to (-34.0, 185.0)
- moved L102 265.2 mm to (-28.0, 182.0)
- moved U102 248.8 mm to (86.0, 228.0)
- moved D104 242.0 mm to (-27.0, 133.0)
- moved D103 238.0 mm to (-38.0, 133.0)
- moved C102 232.9 mm to (7.00, 93.0)
- moved C104 215.5 mm to (25.0, 100.0)
- moved D101 204.8 mm to (40.0, 125.0)
- moved C103 198.9 mm to (35.0, 95.0)
- moved L101 187.1 mm to (35.0, 91.0)
- moved U100 178.3 mm to (22.6, 90.0)
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Connections:
- C102 pad 1: VCOM -> +6V
- C103 pad 1: /[1] Power/BOOST_IN_104 -> VCOM
- C103 pad 2: /[1] Power/SWO_100 -> GND
- C104 pad 1: +3V3 -> /[1] Power/BOOST_IN_104
- C104 pad 2: GND -> /[1] Power/SWO_100
- C106 pad 1: /[1] Power/VBUS1 -> +3V3
- C107 pad 1: +5C -> /[1] Power/VBUS1
- C108 pad 1: /[1] Power/BATT_FILT -> +5C
- C109 pad 1: +3.3VA -> /[1] Power/BATT_FILT
- C110 pad 1: /[1] Power/VBUS2 -> +3.3VA
- C111 pad 1: +5F -> /[1] Power/VBUS2
- C112 pad 1: Net-(C112-Pad1) -> +5F
- C400 pad 1: +3.3VP -> +3V3
- C401 pad 1: +3.3VP -> +3V3
- C402 pad 1: +3.3VP -> +3V3
- C403 pad 1: +3.3VP -> +3V3
- C404 pad 1: +3.3VP -> +3V3
- C407 pad 1: +3.3VP -> +3V3
- C408 pad 1: +3.3VP -> +3V3
- D100 pad 1: VCOM -> /[1] Power/BUCK_OUT_104
- D100 pad 2: +BATT -> GND
- D101 pad 2: +5C -> +BATT
- D102 pad 1: Net-(C112-Pad1) -> VCOM
- D102 pad 2: VCOM -> +5C
- D104 pad 1: Net-(C112-Pad1) -> VCOM
- Q402 pad 1: +3.3VP -> +3V3
- R100 pad 1: VCOM -> /[1] Power/BUCK_FB_104
- R100 pad 2: /[1] Power/BATT_FILT -> +6V
- R101 pad 1: /[1] Power/BUCK_FB_104 -> GND
- R101 pad 2: +6V -> /[1] Power/BUCK_FB_104
- R102 pad 1: GND -> VCOM
- R102 pad 2: /[1] Power/BUCK_FB_104 -> /[1] Power/BATT_FILT
- R404 pad 2: +3.3VP -> +3V3
- R407 pad 1: +3.3VP -> +3V3
- U100 pad 1: +3V3 -> +BATT
- U100 pad 2: VCOM -> /[1] Power/BUCK_OUT_104
- U100 pad 3: VCOM -> GND
- U100 pad 4: GND -> /[1] Power/BUCK_FB_104
- U100 pad 5: /[1] Power/SWO_100 -> GND
- U101 pad 1: GND -> +3V3
- U101 pad 2: +3.3VA -> VCOM
- U101 pad 3: /[1] Power/BATT_FILT -> VCOM
- U102 pad 1: +3.3VP -> GND
- U102 pad 2: Net-(C112-Pad1) -> +3.3VA
- U102 pad 3: Net-(C112-Pad1) -> /[1] Power/BATT_FILT
- U401 pad 16: +3.3VP -> +3V3
- U401 pad 4: +3.3VP -> +3V3
- U402 pad 3: +3.3VP -> +3V3
- U403 pad 10: +3.3VP -> +3V3
