File: PCBs/RCU/ADCs.kicad_sch (KiCad schematic)
At the start: 18 parts, among them U600 ADC121C027CIMK/NOPB, U601 OPA320, U602 ADC121C027CIMK/NOPB, U603 OPA320

Commit message: Wrote slave address for all I2C ICs in binary and hex
Other:
- note added: "Slave Address: 1010000 - 0x50"
- note added: "Slave Address: 1010001 - 0x51"
- note removed: "Slave Address: 1010000"
- note removed: "Slave Address: 1010001"
Changed lines of the file:
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@@
     (effects (font (size 1.27 1.27)) (justify left bottom))
   )
-  (text "Slave Address: 1010001" (at 63.5 55.88 0)
+  (text "Slave Address: 1010001 - 0x51" (at 55.88 58.42 0)
     (effects (font (size 1.27 1.27)) (justify left bottom))
   )
@@
     (effects (font (size 5.08 5.08) (thickness 1.016) bold italic) (justify left bottom))
   )
-  (text "Slave Address: 1010000" (at 63.5 95.25 0)
+  (text "Slave Address: 1010000 - 0x50" (at 55.88 97.79 0)
     (effects (font (size 1.27 1.27)) (justify left bottom))
   )

Commit message: Add footprint to rest of IC's except ESP32
Parts:
- U600, U602: value ADC121C027CIMK/NOPB -> (none)
Changed lines of the file:
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@@
     (in_bom yes) (on_board yes) (fields_autoplaced)
     (property "Reference" "U600" (id 0) (at 74.93 36.83 0))
-    (property "Value" "ADC121C027CIMK/NOPB" (id 1) (at 74.93 39.37 0))
+    (property "Value" "" (id 1) (at 74.93 39.37 0))
     (property "Footprint" "" (id 2) (at 85.09 38.1 0)
       (effects (font (size 1.27 1.27)) hide)
@@
     (in_bom yes) (on_board yes) (fields_autoplaced)
     (property "Reference" "U602" (id 0) (at 74.93 76.2 0))
-    (property "Value" "ADC121C027CIMK/NOPB" (id 1) (at 74.93 78.74 0))
+    (property "Value" "" (id 1) (at 74.93 78.74 0))
     (property "Footprint" "" (id 2) (at 85.09 77.47 0)
       (effects (font (size 1.27 1.27)) hide)

Commit message: Add footprint to power module diodes, and replaced 1N4148W with 2 SM5817's
Parts:
- U600, U602: value (none) -> ADC121C027CIMK/NOPB; footprint (none) -> Package_TO_SOT_SMD:TSOT-23-6
Changed lines of the file:
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@@
     (in_bom yes) (on_board yes) (fields_autoplaced)
     (property "Reference" "U600" (id 0) (at 74.93 36.83 0))
-    (property "Value" "" (id 1) (at 74.93 39.37 0))
-    (property "Footprint" "" (id 2) (at 85.09 38.1 0)
+    (property "Value" "ADC121C027CIMK/NOPB" (id 1) (at 74.93 39.37 0))
+    (property "Footprint" "Package_TO_SOT_SMD:TSOT-23-6" (id 2) (at 85.09 38.1 0)
       (effects (font (size 1.27 1.27)) hide)
     )
@@
     (in_bom yes) (on_board yes) (fields_autoplaced)
     (property "Reference" "U602" (id 0) (at 74.93 76.2 0))
-    (property "Value" "" (id 1) (at 74.93 78.74 0))
-    (property "Footprint" "" (id 2) (at 85.09 77.47 0)
+    (property "Value" "ADC121C027CIMK/NOPB" (id 1) (at 74.93 78.74 0))
+    (property "Footprint" "Package_TO_SOT_SMD:TSOT-23-6" (id 2) (at 85.09 77.47 0)
       (effects (font (size 1.27 1.27)) hide)
     )

Commit message: Add footrpints to TVS diodes in [3]
Parts:
- C600, C602, C604, C605, C607, C609: value 0.1uF -> (none)
- C601, C606: value 10uF -> (none)
- C603, C608: value 1nF -> (none)
- R600, R607: value 15R -> (none)
- R601, R603: value 1.6k -> (none)
- U600, U602: value ADC121C027CIMK/NOPB -> (none); footprint Package_TO_SOT_SMD:TSOT-23-6 -> (none)
- U601, U603: value OPA320 -> (none); footprint Package_TO_SOT_SMD:SOT-23-5 -> (none)

Commit message: Passed ERC
Parts:
- C600, C602, C604, C605, C607, C609: value (none) -> 0.1uF; footprint (none) -> Capacitor_SMD:C_0603_1608Metric
- C601, C606: value (none) -> 10uF; footprint (none) -> Capacitor_SMD:C_0603_1608Metric
- C603, C608: value (none) -> 1nF; footprint (none) -> Capacitor_SMD:C_0603_1608Metric
- R600, R607: value (none) -> 15R; footprint (none) -> Resistor_SMD:R_0603_1608Metric
- R601, R603: value (none) -> 1.6k; footprint (none) -> Resistor_SMD:R_0603_1608Metric
- U600, U602: value (none) -> ADC121C027CIMK/NOPB; footprint (none) -> Package_TO_SOT_SMD:TSOT-23-6
- U601, U603: value (none) -> OPA320; footprint (none) -> Package_TO_SOT_SMD:SOT-23-5
Changed lines of the file:
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@@
       (effects (font (size 1.27 1.27)) (justify left))
     )
-    (property "Value" "" (id 1) (at 139.7 44.45 90)
-      (effects (font (size 1.27 1.27)) (justify left))
-    )
-    (property "Footprint" "" (id 2) (at 138.43 43.688 90)
+    (property "Value" "1.6k" (id 1) (at 139.7 44.45 90)
+      (effects (font (size 1.27 1.27)) (justify left))
+    )
+    (property "Footprint" "Resistor_SMD:R_0603_1608Metric" (id 2) (at 138.43 43.688 90)
       (effects (font (size 1.27 1.27)) hide)
     )
@@
       (effects (font (size 1.27 1.27)) (justify left))
     )
-    (property "Value" "" (id 1) (at 43.18 45.72 0)
-      (effects (font (size 1.27 1.27)) (justify left))
-    )
-    (property "Footprint" "" (id 2) (at 44.7548 48.26 0)
+    (property "Value" "0.1uF" (id 1) (at 43.18 45.72 0)
+      (effects (font (size 1.27 1.27)) (justify left))
+    )
+    (property "Footprint" "Capacitor_SMD:C_0603_1608Metric" (id 2) (at 44.7548 48.26 0)
       (effects (font (size 1.27 1.27)) hide)
     )
@@
       (effects (font (size 1.27 1.27)) (justify right))
     )
-    (property "Value" "" (id 1) (at 135.89 90.1699 0)
-      (effects (font (size 1.27 1.27)) (justify right))
-    )
-    (property "Footprint" "" (id 2) (at 131.1148 85.09 0)
+    (property "Value" "0.1uF" (id 1) (at 135.89 90.1699 0)
+      (effects (font (size 1.27 1.27)) (justify right))
+    )
+    (property "Footprint" "Capacitor_SMD:C_0603_1608Metric" (id 2) (at 131.1148 85.09 0)
       (effects (font (size 1.27 1.27)) hide)
     )
@@
       (effects (font (size 1.27 1.27)) (justify right))
     )
-    (property "Value" "" (id 1) (at 110.49 48.26 0)
-      (effects (font (size 1.27 1.27)) (justify right))
-    )
-    (property "Footprint" "" (id 2) (at 119.38 49.53 0)
+    (property "Value" "OPA320" (id 1) (at 110.49 48.26 0)
+      (effects (font (size 1.27 1.27)) (justify right))
+    )
+    (property "Footprint" "Package_TO_SOT_SMD:SOT-23-5" (id 2) (at 119.38 49.53 0)
       (effects (font (size 1.27 1.27)) (justify left) hide)
     )
@@
     (in_bom yes) (on_board yes)
     (property "Reference" "C600" (id 0) (at 110.49 31.75 90))
-    (property "Value" "" (id 1) (at 110.49 39.37 90))
-    (property "Footprint" "" (id 2) (at 114.3 34.5948 0)
+    (property "Value" "0.1uF" (id 1) (at 110.49 39.37 90))
+    (property "Footprint" "Capacitor_SMD:C_0603_1608Metric" (id 2) (at 114.3 34.5948 0)
       (effects (font (size 1.27 1.27)) hide)
     )
@@
     (in_bom yes) (on_board yes)
     (property "Reference" "C605" (id 0) (at 110.49 71.12 90))
-    (property "Value" "" (id 1) (at 110.49 78.74 90))
-    (property "Footprint" "" (id 2) (at 114.3 73.9648 0)
+    (property "Value" "0.1uF" (id 1) (at 110.49 78.74 90))
+    (property "Footprint" "Capacitor_SMD:C_0603_1608Metric" (id 2) (at 114.3 73.9648 0)
       (effects (font (size 1.27 1.27)) hide)
     )
@@
       (effects (font (size 1.27 1.27)) (justify left))
     )
-    (property "Value" "" (id 1) (at 30.48 45.72 0)
-      (effects (font (size 1.27 1.27)) (justify left))
-    )
-    (property "Footprint" "" (id 2) (at 32.0548 48.26 0)
+    (property "Value" "10uF" (id 1) (at 30.48 45.72 0)
+      (effects (font (size 1.27 1.27)) (justify left))
+    )
+    (property "Footprint" "Capacitor_SMD:C_0603_1608Metric" (id 2) (at 32.0548 48.26 0)
       (effects (font (size 1.27 1.27)) hide)
     )
@@
       (effects (font (size 1.27 1.27)) (justify left))
     )
-    (property "Value" "" (id 1) (at 93.98 95.25 0)
-      (effects (font (size 1.27 1.27)) (justify left))
-    )
-    (property "Footprint" "" (id 2) (at 93.6752 96.52 0)
+    (property "Value" "1nF" (id 1) (at 93.98 95.25 0)
+      (effects (font (size 1.27 1.27)) (justify left))
+    )
+    (property "Footprint" "Capacitor_SMD:C_0603_1608Metric" (id 2) (at 93.6752 96.52 0)
       (effects (font (size 1.27 1.27)) hide)
     )
@@
     (in_bom yes) (on_board yes)
     (property "Reference" "R600" (id 0) (at 99.06 41.91 90))
-    (property "Value" "" (id 1) (at 99.06 46.99 90))
-    (property "Footprint" "" (id 2) (at 99.06 46.228 90)
+    (property "Value" "15R" (id 1) (at 99.06 46.99 90))
+    (property "Footprint" "Resistor_SMD:R_0603_1608Metric" (id 2) (at 99.06 46.228 90)
       (effects (font (size 1.27 1.27)) hide)
     )
@@
       (effects (font (size 1.27 1.27)) (justify left))
     )
-    (property "Value" "" (id 1) (at 93.98 55.88 0)
-      (effects (font (size 1.27 1.27)) (justify left))
-    )
-    (property "Footprint" "" (id 2) (at 93.6752 57.15 0)
+    (property "Value" "1nF" (id 1) (at 93.98 55.88 0)
+      (effects (font (size 1.27 1.27)) (justify left))
+    )
+    (property "Footprint" "Capacitor_SMD:C_0603_1608Metric" (id 2) (at 93.6752 57.15 0)
       (effects (font (size 1.27 1.27)) hide)
     )
@@
       (effects (font (size 1.27 1.27)) (justify left))
     )
-    (property "Value" "" (id 1) (at 30.48 85.09 0)
-      (effects (font (size 1.27 1.27)) (justify left))
-    )
-    (property "Footprint" "" (id 2) (at 32.0548 87.63 0)
+    (property "Value" "10uF" (id 1) (at 30.48 85.09 0)
+      (effects (font (size 1.27 1.27)) (justify left))
+    )
+    (property "Footprint" "Capacitor_SMD:C_0603_1608Metric" (id 2) (at 32.0548 87.63 0)
       (effects (font (size 1.27 1.27)) hide)
     )
@@
       (effects (font (size 1.27 1.27)) (justify left))
     )
-    (property "Value" "" (id 1) (at 43.18 85.09 0)
-      (effects (font (size 1.27 1.27)) (justify left))
-    )
-    (property "Footprint" "" (id 2) (at 44.7548 87.63 0)
+    (property "Value" "0.1uF" (id 1) (at 43.18 85.09 0)
+      (effects (font (size 1.27 1.27)) (justify left))
+    )
+    (property "Footprint" "Capacitor_SMD:C_0603_1608Metric" (id 2) (at 44.7548 87.63 0)
       (effects (font (size 1.27 1.27)) hide)
     )
@@
       (effects (font (size 1.27 1.27)) (justify left))
     )
-    (property "Value" "" (id 1) (at 139.7 83.82 90)
-      (effects (font (size 1.27 1.27)) (justify left))
-    )
-    (property "Footprint" "" (id 2) (at 138.43 83.058 90)
+    (property "Value" "1.6k" (id 1) (at 139.7 83.82 90)
+      (effects (font (size 1.27 1.27)) (justify left))
+    )
+    (property "Footprint" "Resistor_SMD:R_0603_1608Metric" (id 2) (at 138.43 83.058 90)
       (effects (font (size 1.27 1.27)) hide)
     )
@@
     (in_bom yes) (on_board yes) (fields_autoplaced)
     (property "Reference" "U600" (id 0) (at 74.93 36.83 0))
-    (property "Value" "" (id 1) (at 74.93 39.37 0))
-    (property "Footprint" "" (id 2) (at 85.09 38.1 0)
+    (property "Value" "ADC121C027CIMK/NOPB" (id 1) (at 74.93 39.37 0))
+    (property "Footprint" "Package_TO_SOT_SMD:TSOT-23-6" (id 2) (at 85.09 38.1 0)
       (effects (font (size 1.27 1.27)) hide)
     )
@@
       (effects (font (size 1.27 1.27)) (justify right))
     )
-    (property "Value" "" (id 1) (at 110.49 87.63 0)
-      (effects (font (size 1.27 1.27)) (justify right))
-    )
-    (property "Footprint" "" (id 2) (at 119.38 88.9 0)
+    (property "Value" "OPA320" (id 1) (at 110.49 87.63 0)
+      (effects (font (size 1.27 1.27)) (justify right))
+    )
+    (property "Footprint" "Package_TO_SOT_SMD:SOT-23-5" (id 2) (at 119.38 88.9 0)
       (effects (font (size 1.27 1.27)) (justify left) hide)
     )
@@
       (effects (font (size 1.27 1.27)) (justify right))
     )
-    (property "Value" "" (id 1) (at 135.89 50.7999 0)
-      (effects (font (size 1.27 1.27)) (justify right))
-    )
-    (property "Footprint" "" (id 2) (at 131.1148 45.72 0)
+    (property "Value" "0.1uF" (id 1) (at 135.89 50.7999 0)
+      (effects (font (size 1.27 1.27)) (justify right))
+    )
+    (property "Footprint" "Capacitor_SMD:C_0603_1608Metric" (id 2) (at 131.1148 45.72 0)
       (effects (font (size 1.27 1.27)) hide)
     )
@@
     (in_bom yes) (on_board yes)
     (property "Reference" "R607" (id 0) (at 99.06 81.28 90))
-    (property "Value" "" (id 1) (at 99.06 86.36 90))
-    (property "Footprint" "" (id 2) (at 99.06 85.598 90)
+    (property "Value" "15R" (id 1) (at 99.06 86.36 90))
+    (property "Footprint" "Resistor_SMD:R_0603_1608Metric" (id 2) (at 99.06 85.598 90)
       (effects (font (size 1.27 1.27)) hide)
     )
@@
     (in_bom yes) (on_board yes) (fields_autoplaced)
     (property "Reference" "U602" (id 0) (at 74.93 76.2 0))
-    (property "Value" "" (id 1) (at 74.93 78.74 0))
-    (property "Footprint" "" (id 2) (at 85.09 77.47 0)
-      (effects (font (size 1.27 1.27)) hide)
-    )
+    (property "Value" "ADC121C027CIMK/NOPB" (id 1) (at 74.93 78.74 0))
+    (property "Footprint" "Package_TO_SOT_SMD:TSOT-23-6" (id 2) (at 85.09 77.47 0)
+      (effects (font (size 1.27 1.27)) hide)
+    )

Commit message: Finished routing 3.3V regulator
Parts:
- C600, C602, C605, C607: value 0.1uF -> (none); footprint Capacitor_SMD:C_0603_1608Metric -> (none)
- C601, C606: value 10uF -> (none); footprint Capacitor_SMD:C_0603_1608Metric -> (none)
- C603, C608: value 1nF -> (none); footprint Capacitor_SMD:C_0603_1608Metric -> (none)
- R600, R607: value 15R -> (none); footprint Resistor_SMD:R_0603_1608Metric -> (none)
Changed lines of the file:
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@@
       (effects (font (size 1.27 1.27)) (justify left))
     )
-    (property "Value" "0.1uF" (id 1) (at 43.18 45.72 0)
-      (effects (font (size 1.27 1.27)) (justify left))
-    )
-    (property "Footprint" "Capacitor_SMD:C_0603_1608Metric" (id 2) (at 44.7548 48.26 0)
+    (property "Value" "" (id 1) (at 43.18 45.72 0)
+      (effects (font (size 1.27 1.27)) (justify left))
+    )
+    (property "Footprint" "" (id 2) (at 44.7548 48.26 0)
       (effects (font (size 1.27 1.27)) hide)
     )
@@
     (in_bom yes) (on_board yes)
     (property "Reference" "C600" (id 0) (at 110.49 31.75 90))
-    (property "Value" "0.1uF" (id 1) (at 110.49 39.37 90))
-    (property "Footprint" "Capacitor_SMD:C_0603_1608Metric" (id 2) (at 114.3 34.5948 0)
+    (property "Value" "" (id 1) (at 110.49 39.37 90))
+    (property "Footprint" "" (id 2) (at 114.3 34.5948 0)
       (effects (font (size 1.27 1.27)) hide)
     )
@@
     (in_bom yes) (on_board yes)
     (property "Reference" "C605" (id 0) (at 110.49 71.12 90))
-    (property "Value" "0.1uF" (id 1) (at 110.49 78.74 90))
-    (property "Footprint" "Capacitor_SMD:C_0603_1608Metric" (id 2) (at 114.3 73.9648 0)
+    (property "Value" "" (id 1) (at 110.49 78.74 90))
+    (property "Footprint" "" (id 2) (at 114.3 73.9648 0)
       (effects (font (size 1.27 1.27)) hide)
     )
@@
       (effects (font (size 1.27 1.27)) (justify left))
     )
-    (property "Value" "10uF" (id 1) (at 30.48 45.72 0)
-      (effects (font (size 1.27 1.27)) (justify left))
-    )
-    (property "Footprint" "Capacitor_SMD:C_0603_1608Metric" (id 2) (at 32.0548 48.26 0)
+    (property "Value" "" (id 1) (at 30.48 45.72 0)
+      (effects (font (size 1.27 1.27)) (justify left))
+    )
+    (property "Footprint" "" (id 2) (at 32.0548 48.26 0)
       (effects (font (size 1.27 1.27)) hide)
     )
@@
       (effects (font (size 1.27 1.27)) (justify left))
     )
-    (property "Value" "1nF" (id 1) (at 93.98 95.25 0)
-      (effects (font (size 1.27 1.27)) (justify left))
-    )
-    (property "Footprint" "Capacitor_SMD:C_0603_1608Metric" (id 2) (at 93.6752 96.52 0)
+    (property "Value" "" (id 1) (at 93.98 95.25 0)
+      (effects (font (size 1.27 1.27)) (justify left))
+    )
+    (property "Footprint" "" (id 2) (at 93.6752 96.52 0)
       (effects (font (size 1.27 1.27)) hide)
     )
@@
     (in_bom yes) (on_board yes)
     (property "Reference" "R600" (id 0) (at 99.06 41.91 90))
-    (property "Value" "15R" (id 1) (at 99.06 46.99 90))
-    (property "Footprint" "Resistor_SMD:R_0603_1608Metric" (id 2) (at 99.06 46.228 90)
+    (property "Value" "" (id 1) (at 99.06 46.99 90))
+    (property "Footprint" "" (id 2) (at 99.06 46.228 90)
       (effects (font (size 1.27 1.27)) hide)
     )
@@
       (effects (font (size 1.27 1.27)) (justify left))
     )
-    (property "Value" "1nF" (id 1) (at 93.98 55.88 0)
-      (effects (font (size 1.27 1.27)) (justify left))
-    )
-    (property "Footprint" "Capacitor_SMD:C_0603_1608Metric" (id 2) (at 93.6752 57.15 0)
+    (property "Value" "" (id 1) (at 93.98 55.88 0)
+      (effects (font (size 1.27 1.27)) (justify left))
+    )
+    (property "Footprint" "" (id 2) (at 93.6752 57.15 0)
       (effects (font (size 1.27 1.27)) hide)
     )
@@
       (effects (font (size 1.27 1.27)) (justify left))
     )
-    (property "Value" "10uF" (id 1) (at 30.48 85.09 0)
-      (effects (font (size 1.27 1.27)) (justify left))
-    )
-    (property "Footprint" "Capacitor_SMD:C_0603_1608Metric" (id 2) (at 32.0548 87.63 0)
+    (property "Value" "" (id 1) (at 30.48 85.09 0)
+      (effects (font (size 1.27 1.27)) (justify left))
+    )
+    (property "Footprint" "" (id 2) (at 32.0548 87.63 0)
       (effects (font (size 1.27 1.27)) hide)
     )
@@
       (effects (font (size 1.27 1.27)) (justify left))
     )
-    (property "Value" "0.1uF" (id 1) (at 43.18 85.09 0)
-      (effects (font (size 1.27 1.27)) (justify left))
-    )
-    (property "Footprint" "Capacitor_SMD:C_0603_1608Metric" (id 2) (at 44.7548 87.63 0)
+    (property "Value" "" (id 1) (at 43.18 85.09 0)
+      (effects (font (size 1.27 1.27)) (justify left))
+    )
+    (property "Footprint" "" (id 2) (at 44.7548 87.63 0)
       (effects (font (size 1.27 1.27)) hide)
     )
@@
     (in_bom yes) (on_board yes)
     (property "Reference" "R607" (id 0) (at 99.06 81.28 90))
-    (property "Value" "15R" (id 1) (at 99.06 86.36 90))
-    (property "Footprint" "Resistor_SMD:R_0603_1608Metric" (id 2) (at 99.06 85.598 90)
-      (effects (font (size 1.27 1.27)) hide)
-    )
+    (property "Value" "" (id 1) (at 99.06 86.36 90))
+    (property "Footprint" "" (id 2) (at 99.06 85.598 90)
+      (effects (font (size 1.27 1.27)) hide)
+    )

Commit message: Traced I2C lines
Parts:
- C600, C602, C605, C607: value (none) -> 0.1uF; footprint (none) -> Capacitor_SMD:C_0402_1005Metric
- C601, C606: value (none) -> 10uF; footprint (none) -> Capacitor_SMD:C_0402_1005Metric
- C603, C608: value (none) -> 1nF; footprint (none) -> Capacitor_SMD:C_0402_1005Metric
- R600, R607: value (none) -> 15R; footprint (none) -> Resistor_SMD:R_0402_1005Metric
Changed lines of the file:
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@@
       (effects (font (size 1.27 1.27)) (justify left))
     )
-    (property "Value" "" (id 1) (at 43.18 45.72 0)
-      (effects (font (size 1.27 1.27)) (justify left))
-    )
-    (property "Footprint" "" (id 2) (at 44.7548 48.26 0)
+    (property "Value" "0.1uF" (id 1) (at 43.18 45.72 0)
+      (effects (font (size 1.27 1.27)) (justify left))
+    )
+    (property "Footprint" "Capacitor_SMD:C_0402_1005Metric" (id 2) (at 44.7548 48.26 0)
       (effects (font (size 1.27 1.27)) hide)
     )
@@
     (in_bom yes) (on_board yes)
     (property "Reference" "C600" (id 0) (at 110.49 31.75 90))
-    (property "Value" "" (id 1) (at 110.49 39.37 90))
-    (property "Footprint" "" (id 2) (at 114.3 34.5948 0)
+    (property "Value" "0.1uF" (id 1) (at 110.49 39.37 90))
+    (property "Footprint" "Capacitor_SMD:C_0402_1005Metric" (id 2) (at 114.3 34.5948 0)
       (effects (font (size 1.27 1.27)) hide)
     )
@@
     (in_bom yes) (on_board yes)
     (property "Reference" "C605" (id 0) (at 110.49 71.12 90))
-    (property "Value" "" (id 1) (at 110.49 78.74 90))
-    (property "Footprint" "" (id 2) (at 114.3 73.9648 0)
+    (property "Value" "0.1uF" (id 1) (at 110.49 78.74 90))
+    (property "Footprint" "Capacitor_SMD:C_0402_1005Metric" (id 2) (at 114.3 73.9648 0)
       (effects (font (size 1.27 1.27)) hide)
     )
@@
       (effects (font (size 1.27 1.27)) (justify left))
     )
-    (property "Value" "" (id 1) (at 30.48 45.72 0)
-      (effects (font (size 1.27 1.27)) (justify left))
-    )
-    (property "Footprint" "" (id 2) (at 32.0548 48.26 0)
+    (property "Value" "10uF" (id 1) (at 30.48 45.72 0)
+      (effects (font (size 1.27 1.27)) (justify left))
+    )
+    (property "Footprint" "Capacitor_SMD:C_0402_1005Metric" (id 2) (at 32.0548 48.26 0)
       (effects (font (size 1.27 1.27)) hide)
     )
@@
       (effects (font (size 1.27 1.27)) (justify left))
     )
-    (property "Value" "" (id 1) (at 93.98 95.25 0)
-      (effects (font (size 1.27 1.27)) (justify left))
-    )
-    (property "Footprint" "" (id 2) (at 93.6752 96.52 0)
+    (property "Value" "1nF" (id 1) (at 93.98 95.25 0)
+      (effects (font (size 1.27 1.27)) (justify left))
+    )
+    (property "Footprint" "Capacitor_SMD:C_0402_1005Metric" (id 2) (at 93.6752 96.52 0)
       (effects (font (size 1.27 1.27)) hide)
     )
@@
     (in_bom yes) (on_board yes)
     (property "Reference" "R600" (id 0) (at 99.06 41.91 90))
-    (property "Value" "" (id 1) (at 99.06 46.99 90))
-    (property "Footprint" "" (id 2) (at 99.06 46.228 90)
+    (property "Value" "15R" (id 1) (at 99.06 46.99 90))
+    (property "Footprint" "Resistor_SMD:R_0402_1005Metric" (id 2) (at 99.06 46.228 90)
       (effects (font (size 1.27 1.27)) hide)
     )
@@
       (effects (font (size 1.27 1.27)) (justify left))
     )
-    (property "Value" "" (id 1) (at 93.98 55.88 0)
-      (effects (font (size 1.27 1.27)) (justify left))
-    )
-    (property "Footprint" "" (id 2) (at 93.6752 57.15 0)
+    (property "Value" "1nF" (id 1) (at 93.98 55.88 0)
+      (effects (font (size 1.27 1.27)) (justify left))
+    )
+    (property "Footprint" "Capacitor_SMD:C_0402_1005Metric" (id 2) (at 93.6752 57.15 0)
       (effects (font (size 1.27 1.27)) hide)
     )
@@
       (effects (font (size 1.27 1.27)) (justify left))
     )
-    (property "Value" "" (id 1) (at 30.48 85.09 0)
-      (effects (font (size 1.27 1.27)) (justify left))
-    )
-    (property "Footprint" "" (id 2) (at 32.0548 87.63 0)
+    (property "Value" "10uF" (id 1) (at 30.48 85.09 0)
+      (effects (font (size 1.27 1.27)) (justify left))
+    )
+    (property "Footprint" "Capacitor_SMD:C_0402_1005Metric" (id 2) (at 32.0548 87.63 0)
       (effects (font (size 1.27 1.27)) hide)
     )
@@
       (effects (font (size 1.27 1.27)) (justify left))
     )
-    (property "Value" "" (id 1) (at 43.18 85.09 0)
-      (effects (font (size 1.27 1.27)) (justify left))
-    )
-    (property "Footprint" "" (id 2) (at 44.7548 87.63 0)
+    (property "Value" "0.1uF" (id 1) (at 43.18 85.09 0)
+      (effects (font (size 1.27 1.27)) (justify left))
+    )
+    (property "Footprint" "Capacitor_SMD:C_0402_1005Metric" (id 2) (at 44.7548 87.63 0)
       (effects (font (size 1.27 1.27)) hide)
     )
@@
     (in_bom yes) (on_board yes)
     (property "Reference" "R607" (id 0) (at 99.06 81.28 90))
-    (property "Value" "" (id 1) (at 99.06 86.36 90))
-    (property "Footprint" "" (id 2) (at 99.06 85.598 90)
-      (effects (font (size 1.27 1.27)) hide)
-    )
+    (property "Value" "15R" (id 1) (at 99.06 86.36 90))
+    (property "Footprint" "Resistor_SMD:R_0402_1005Metric" (id 2) (at 99.06 85.598 90)
+      (effects (font (size 1.27 1.27)) hide)
+    )
