File: PCBs/RCU/external_memory.kicad_sch (KiCad schematic)
At the start: 2 parts

Commit message: Passed ERC
Parts:
- C700: value (none) -> 1uF; footprint (none) -> Capacitor_SMD:C_0603_1608Metric
- U700: value (none) -> SST26VF032BT-104I/SM; footprint (none) -> Package_SO:SOIC-8_5.275x5.275mm_P1.27mm
Changed lines of the file:
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@@
       (effects (font (size 1.27 1.27)) (justify left))
     )
-    (property "Value" "" (id 1) (at 127 71.1199 0)
+    (property "Value" "1uF" (id 1) (at 127 71.1199 0)
       (effects (font (size 1.27 1.27)) (justify left))
     )
-    (property "Footprint" "" (id 2) (at 124.1552 73.66 0)
+    (property "Footprint" "Capacitor_SMD:C_0603_1608Metric" (id 2) (at 124.1552 73.66 0)
       (effects (font (size 1.27 1.27)) hide)
     )
@@
     (in_bom yes) (on_board yes)
     (property "Reference" "U700" (id 0) (at 93.98 78.74 0))
-    (property "Value" "" (id 1) (at 76.2 81.28 0))
-    (property "Footprint" "" (id 2) (at 90.17 87.63 0)
+    (property "Value" "SST26VF032BT-104I/SM" (id 1) (at 76.2 81.28 0))
+    (property "Footprint" "Package_SO:SOIC-8_5.275x5.275mm_P1.27mm" (id 2) (at 90.17 87.63 0)
       (effects (font (size 1.27 1.27)) hide)
     )

Commit message: Changed priority of non-ground copper pours to 1
Connections:
- net +3V3: now also C700.2; no longer C700.1
- net GND: now also C700.1; no longer C700.2
Other:
- moved on the sheet: C700
Changed lines of the file:
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@@
     (pin "1")
   )
-  (symbol (lib_id "Device:C") (at 123.19 69.85 0) (unit 1)
+  (symbol (lib_id "Device:C") (at 123.19 69.85 180) (unit 1)
     (in_bom yes) (on_board yes) (fields_autoplaced)
     (property "Reference" "C700" (id 0) (at 127 68.5799 0)
-      (effects (font (size 1.27 1.27)) (justify left))
+      (effects (font (size 1.27 1.27)) (justify right))
     )
     (property "Value" "1uF" (id 1) (at 127 71.1199 0)
-      (effects (font (size 1.27 1.27)) (justify left))
+      (effects (font (size 1.27 1.27)) (justify right))
     )
-    (property "Footprint" "Capacitor_SMD:C_0603_1608Metric" (id 2) (at 124.1552 73.66 0)
+    (property "Footprint" "Capacitor_SMD:C_0603_1608Metric" (id 2) (at 122.2248 66.04 0)
       (effects (font (size 1.27 1.27)) hide)
     )
