File: PCBs/KiCad/RCU/Power.kicad_sch (KiCad schematic)
At the start: 29 parts, among them J100 Conn_01x02, U100 LM2576S-ADJ, U101 AP63203WU, U102 AZ1117-3.3

Commit message: Moved project library one folder up to Kicad Folder
Parts:
- R100: value (none) -> 5.9k; footprint (none) -> Resistor_SMD:R_0603_1608Metric
