File: PCBs/KiCad/RCU/bluetooth.kicad_sch (KiCad schematic)
At the start: 31 parts, among them J400 USB_C_Receptacle_USB2.0, Q400 2N7002NXAKR (NMOS), Q401 2N7002NXAKR (NMOS), Q402 BSS84AK,215 (PMOS), Q403 2N7002NXAKR (NMOS), SW400 SW_Push, SW401 SW_SPDT, U400 USBLC6-2SC6, U401 CH340C, U402 ESP32-MINI-1, U403 DG2788ADN-T1-GE4

Commit message: Moved project library one folder up to Kicad Folder
Parts:
- removed U402: ESP32-MINI-1, ESP32_MINI:XCVR_ESP32-MINI-1-N4, symbol Ghanis_Symbols_KiCad6:ESP32-MINI-1
- added U402: ESP32-C3-MINI-1, ESP32-MINI-1-N4:XCVR_ESP32-MINI-1-N4, symbol ESP32-C3-MINI-1:ESP32-C3-MINI-1
Connections:
- net +3V3: now also U402.3 (3V3)
- net BT_EN: now also U402.8 (EN)
- net GND: now also U402.1 (GND), U402.2 (GND), U402.27 (GND), U402.38 (GND), U402.39 (GND), U402.40 (GND), U402.41 (GND), U402.42 (GND), U402.43 (GND), U402.44 (GND), U402.45 (GND), U402.46 (GND), U402.47 (GND), U402.48 (GND), U402.49 (GND), U402.50 (GND), U402.51 (GND), U402.52 (GND), U402.53 (GND), U402.54 (GND), U402.55 (GND)
- net IO0: now also U402.21 (IO0)
- net UART_BT_RX: now also U402.35 (RXD0)
- net UART_BT_TX: now also U402.36 (TXD0)
