File: PCBs/KiCad/Remote_Controller/Power.kicad_sch (KiCad schematic)
At the start: 29 parts, among them Q101 IRF7319, Q102 IRFML8244TRPBF, Q103 IRFML8244TRPBF, SW101 Power Switch, U101 AP63203WU, U102 LM74700, U103 MCP1700T-3002E/TT, U104 LM74700

Commit message: Added new symbol fields and completed BOM
Parts:
- BT101: Manufacturer Part # (none) -> BA9VPC
- C101, C106, C108, C111, C113: JLCPCB Part # (none) -> C155422; Manufacturer Part # (none) -> CL05B104KA5NNNC
- C102, C109, C110: JLCPCB Part # (none) -> C14445; Manufacturer Part # (none) -> CL05A105KP5NNNC
- C103: JLCPCB Part # (none) -> C84416; Manufacturer Part # (none) -> GRM21BR61E106KA73L
- C104, C105, C107, C112: JLCPCB Part # (none) -> C77091; Manufacturer Part # (none) -> GRM31CR61E226KE15L
- D101: JLCPCB Part # (none) -> C320520; Manufacturer Part # (none) -> P6SMB22CA
- D102: JLCPCB Part # (none) -> C5252984; Manufacturer Part # (none) -> 150060GS75000
- L101: JLCPCB Part # (none) -> C257229; Manufacturer Part # (none) -> SQH6012S-4R0N-LF
- Q101: JLCPCB Part # (none) -> C2760082; Manufacturer Part # (none) -> IRF7319TRPBF
- Q102, Q103: JLCPCB Part # (none) -> C5381404; Manufacturer Part # (none) -> IRFML8244TRPBF
- R101, R102: JLCPCB Part # (none) -> C25531; Manufacturer Part # (none) -> 0402WGJ0103TCE
- R103: JLCPCB Part # (none) -> C14675; Manufacturer Part # (none) -> RC0603FR-07100KL
- R104: value 160R -> 200R; JLCPCB Part # (none) -> C8218; Manufacturer Part # (none) -> 0603WAF2000T5E
- SW101: JLCPCB Part # (none) -> C455234; Manufacturer Part # (none) -> TS-1003ST-26
- U101: JLCPCB Part # (none) -> AP63203WU-7; Manufacturer Part # (none) -> C780769
- U102, U104: JLCPCB Part # (none) -> C2941042; Manufacturer Part # (none) -> LM74700QDBVRQ1
- U103: JLCPCB Part # (none) -> C62244; Manufacturer Part # (none) -> MCP1700T-3002E/TT

Commit message: Added silkscreen text and made manufacturing files
Other:
- title: (none) -> SurvBot - Remote Controller
Changed lines of the file:
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@@
 	(generator_version "8.0")
 	(paper "A4")
+	(title_block
+		(title "SurvBot - Remote Controller")
+		(date "2025-03-17")
+		(rev "1.0.0.")
+	)
 	(junction
 		(at 59.69 109.22)
